Commit message: fixed spawning issue with husky robot

File: src/eecs256aw25/models/husky_description/urdf/husky.urdf.xacro (robot description, xacro)
@@ -10,34 +10,10 @@
   <xacro:if value="$(arg is_sim)">
     <gazebo>
-      <plugin name="$(arg prefix)gazebo_ros2_control" filename="libgazebo_ros2_control.so">
+      <plugin name="gz_ros2_control::GazeboSimROS2ControlPlugin" filename="libgz_ros2_control-system.so">
         <parameters>$(arg gazebo_controllers)</parameters>
       </plugin>
     </gazebo>
-    <gazebo reference="$(arg prefix)imu_link">
-      <sensor name="$(arg prefix)imu_sensor" type="imu">
-      <plugin filename="libgazebo_ros_imu_sensor.so" name="$(arg prefix)imu_plugin">
-          <ros>
-            <namespace>$(arg prefix)</namespace>
-            <remapping>~/out:=imu/data_raw</remapping>
-          </ros>
-          <initial_orientation_as_reference>false</initial_orientation_as_reference>
-        </plugin>
-        <always_on>true</always_on>
-        <update_rate>100</update_rate>
-        <visualize>true</visualize>
-      </sensor>
-    </gazebo>
-    <gazebo reference="$(arg prefix)gps_link">
-      <sensor name="$(arg prefix)gps_sensor" type="gps">
-      <plugin filename="libgazebo_ros_gps_sensor.so" name="$(arg prefix)gps_plugin">
-          <ros>
-            <namespace>$(arg prefix)</namespace>
-            <remapping>~/out:=gps/data</remapping>
-          </ros>
-        </plugin>
-        <always_on>true</always_on>
-        <update_rate>10</update_rate>
-      </sensor>
-    </gazebo>
+    <!-- IMU and GPS disabled for Gazebo Sim migration (Classic plugins removed) -->
+    <!-- Use ros_gz_bridge to expose sensor data if needed -->
   </xacro:if>
   <!-- Optional custom includes. -->

File: src/eecs256aw25/models/husky_description/urdf/husky_macro.urdf.xacro (robot description, xacro)
@@ -136,5 +136,5 @@
       <hardware>
         <xacro:if value="$(arg is_sim)">
-          <plugin>gazebo_ros2_control/GazeboSystem</plugin>
+          <plugin>gz_ros2_control/GazeboSimSystem</plugin>
         </xacro:if>
         <xacro:unless value="$(arg is_sim)">

File: src/eecs256aw25/models/husky_ur_extras.urdf.xacro (robot description, xacro)
@@ -17,5 +17,9 @@
     visual_parameters_file="$(find eecs256aw25)/models/ur_description/config/ur5/visual_parameters.yaml"
     >
-    <origin xyz="$(arg arm_xyz)" rpy="$(arg arm_rpy)"/>
+    <origin xyz="-0.105 0.0 0.0" rpy="0 0 0"/>
   </xacro:ur_robot>
+  <!-- Include UR ros2_control macro -->
+  <xacro:include filename="$(find eecs256aw25)/models/ur_description/urdf/ur_gz.ros2_control.xacro"/>
+  <!-- Instantiate the UR ros2_control macro -->
+  <xacro:ur_ros2_control name="ur" prefix="ur_arm_"/>
 </robot>
